File: PCB/ethernet.kicad_sch (KiCad schematic)
At the start: 21 parts, among them J3 74984104400, U5 LAN8720A, Y2 ECS-250-20-33-CKM-TR

Commit message: Started on board layout
Parts:
- C12, C13, C14, C15, C16, C17, C18: footprint (none) -> Capacitor_SMD:C_0805_2012Metric
- J3: footprint Connector_RJ:RJ45_UDE_RB1-125B8G1A -> ProjectFootprints:74984104400
- L4, L5: footprint (none) -> Inductor_SMD:L_0805_2012Metric
- R10, R11, R12, R13, R14, R5, R6, R8, R9: footprint (none) -> Resistor_SMD:R_0805_2012Metric
- Y2: footprint (none) -> Crystal:Crystal_SMD_3225-4Pin_3.2x2.5mm
Connections:
- net ETH_RX+: now also U5.21 (TXP); no longer U5.23 (RXP)
- net ETH_RX-: now also U5.20 (TXN); no longer U5.22 (RXN)
- net ETH_TX+: now also U5.23 (RXP); no longer U5.21 (TXP)
- net ETH_TX-: now also U5.22 (RXN); no longer U5.20 (TXN)
Changed lines of the file:
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@@
   (junction (at 218.44 123.19) (diameter 0) (color 0 0 0 0)
   )
+  (junction (at 113.03 113.03) (diameter 0) (color 0 0 0 0)
+  )
+  (junction (at 101.6 83.82) (diameter 0) (color 0 0 0 0)
+  )
+  (junction (at 105.41 105.41) (diameter 0) (color 0 0 0 0)
+  )
+  (junction (at 82.55 77.47) (diameter 0) (color 0 0 0 0)
+  )
+  (junction (at 140.97 77.47) (diameter 0) (color 0 0 0 0)
+  )
+  (junction (at 213.36 125.73) (diameter 0) (color 0 0 0 0)
+  )
+  (junction (at 113.03 83.82) (diameter 0) (color 0 0 0 0)
+  )
   (junction (at 101.6 100.33) (diameter 0) (color 0 0 0 0)
-  )
-  (junction (at 113.03 113.03) (diameter 0) (color 0 0 0 0)
-  )
-  (junction (at 101.6 83.82) (diameter 0) (color 0 0 0 0)
-  )
-  (junction (at 105.41 105.41) (diameter 0) (color 0 0 0 0)
-  )
-  (junction (at 82.55 77.47) (diameter 0) (color 0 0 0 0)
-  )
-  (junction (at 140.97 77.47) (diameter 0) (color 0 0 0 0)
-  )
-  (junction (at 213.36 125.73) (diameter 0) (color 0 0 0 0)
-  )
-  (junction (at 113.03 83.82) (diameter 0) (color 0 0 0 0)
   )
   (junction (at 205.74 130.81) (diameter 0) (color 0 0 0 0)
@@
     (stroke (width 0) (type default))
   )
+  (wire (pts (xy 147.32 107.95) (xy 157.48 107.95))
+    (stroke (width 0) (type default))
+  )
   (wire (pts (xy 105.41 92.71) (xy 105.41 105.41))
     (stroke (width 0) (type default))
@@
     (stroke (width 0) (type default))
   )
-  (wire (pts (xy 115.57 102.87) (xy 157.48 102.87))
-    (stroke (width 0) (type default))
-  )
   (wire (pts (xy 213.36 118.11) (xy 213.36 125.73))
     (stroke (width 0) (type default))
@@
     (stroke (width 0) (type default))
   )
-  (wire (pts (xy 116.84 105.41) (xy 157.48 105.41))
+  (wire (pts (xy 142.24 102.87) (xy 147.32 107.95))
     (stroke (width 0) (type default))
   )
@@
     (stroke (width 0) (type default))
   )
+  (wire (pts (xy 143.51 107.95) (xy 148.59 102.87))
+    (stroke (width 0) (type default))
+  )
   (wire (pts (xy 198.12 105.41) (xy 195.58 105.41))
     (stroke (width 0) (type default))
   )
+  (wire (pts (xy 148.59 100.33) (xy 157.48 100.33))
+    (stroke (width 0) (type default))
+  )
   (wire (pts (xy 105.41 83.82) (xy 105.41 85.09))
     (stroke (width 0) (type default))
   )
+  (wire (pts (xy 101.6 100.33) (xy 142.24 100.33))
+    (stroke (width 0) (type default))
+  )
   (wire (pts (xy 105.41 105.41) (xy 96.52 105.41))
     (stroke (width 0) (type default))
@@
     (stroke (width 0) (type default))
   )
+  (wire (pts (xy 115.57 102.87) (xy 142.24 102.87))
+    (stroke (width 0) (type default))
+  )
+  (wire (pts (xy 143.51 105.41) (xy 148.59 100.33))
+    (stroke (width 0) (type default))
+  )
   (wire (pts (xy 214.63 138.43) (xy 205.74 138.43))
     (stroke (width 0) (type default))
@@
     (stroke (width 0) (type default))
   )
+  (wire (pts (xy 116.84 105.41) (xy 143.51 105.41))
+    (stroke (width 0) (type default))
+  )
   (wire (pts (xy 119.38 83.82) (xy 113.03 83.82))
     (stroke (width 0) (type default))
@@
     (stroke (width 0) (type default))
   )
+  (wire (pts (xy 142.24 100.33) (xy 147.32 105.41))
+    (stroke (width 0) (type default))
+  )
   (wire (pts (xy 175.26 66.04) (xy 175.26 67.31))
     (stroke (width 0) (type default))
@@
     (stroke (width 0) (type default))
   )
-  (wire (pts (xy 118.11 107.95) (xy 157.48 107.95))
-    (stroke (width 0) (type default))
-  )
   (wire (pts (xy 210.82 146.05) (xy 200.66 146.05))
     (stroke (width 0) (type default))
@@
     (stroke (width 0) (type default))
   )
-  (wire (pts (xy 101.6 100.33) (xy 157.48 100.33))
-    (stroke (width 0) (type default))
-  )
   (wire (pts (xy 222.25 130.81) (xy 222.25 138.43))
     (stroke (width 0) (type default))
@@
     (stroke (width 0) (type default))
   )
+  (wire (pts (xy 147.32 105.41) (xy 157.48 105.41))
+    (stroke (width 0) (type default))
+  )
   (wire (pts (xy 213.36 109.22) (xy 213.36 110.49))
     (stroke (width 0) (type default))
@@
     (stroke (width 0) (type default))
   )
+  (wire (pts (xy 118.11 107.95) (xy 143.51 107.95))
+    (stroke (width 0) (type default))
+  )
   (wire (pts (xy 198.12 110.49) (xy 195.58 110.49))
     (stroke (width 0) (type default))
@@
   )
   (wire (pts (xy 152.4 125.73) (xy 152.4 115.57))
+    (stroke (width 0) (type default))
+  )
+  (wire (pts (xy 148.59 102.87) (xy 157.48 102.87))
     (stroke (width 0) (type default))
   )
@@
       (effects (font (size 1.27 1.27)) (justify right))
     )
-    (property "Footprint" "" (at 205.74 134.62 0)
+    (property "Footprint" "Crystal:Crystal_SMD_3225-4Pin_3.2x2.5mm" (at 205.74 134.62 0)
       (effects (font (size 1.27 1.27)) hide)
     )
@@
       (effects (font (size 1.27 1.27)) (justify right))
     )
-    (property "Footprint" "" (at 113.03 78.74 0)
+    (property "Footprint" "Inductor_SMD:L_0805_2012Metric" (at 113.03 78.74 0)
       (effects (font (size 1.27 1.27)) hide)
     )
@@
       (effects (font (size 1.27 1.27)) (justify right))
     )
-    (property "Footprint" "" (at 175.26 71.12 0)
+    (property "Footprint" "Inductor_SMD:L_0805_2012Metric" (at 175.26 71.12 0)
       (effects (font (size 1.27 1.27)) hide)
     )
@@
       (effects (font (size 1.27 1.27)))
     )
-    (property "Footprint" "" (at 80.518 83.82 90)
+    (property "Footprint" "Resistor_SMD:R_0805_2012Metric" (at 80.518 83.82 90)
       (effects (font (size 1.27 1.27)) hide)
     )
@@
       (effects (font (size 1.27 1.27)) (justify left))
     )
-    (property "Footprint" "Connector_RJ:RJ45_UDE_RB1-125B8G1A" (at 83.82 74.93 0)
+    (property "Footprint" "ProjectFootprints:74984104400" (at 83.82 74.93 0)
       (effects (font (size 1.27 1.27)) hide)
     )
@@
       (effects (font (size 1.27 1.27)) (justify left))
     )
-    (property "Footprint" "" (at 118.4148 92.71 0)
+    (property "Footprint" "Capacitor_SMD:C_0805_2012Metric" (at 118.4148 92.71 0)
       (effects (font (size 1.27 1.27)) hide)
     )
@@
       (effects (font (size 1.27 1.27)))
     )
-    (property "Footprint" "" (at 114.808 88.9 90)
+    (property "Footprint" "Resistor_SMD:R_0805_2012Metric" (at 114.808 88.9 90)
       (effects (font (size 1.27 1.27)) hide)
     )
@@
       (effects (font (size 1.27 1.27)) (justify left))
     )
-    (property "Footprint" "" (at 215.5952 138.43 0)
+    (property "Footprint" "Capacitor_SMD:C_0805_2012Metric" (at 215.5952 138.43 0)
       (effects (font (size 1.27 1.27)) hide)
     )
@@
       (effects (font (size 1.27 1.27)) (justify left))
     )
-    (property "Footprint" "" (at 154.178 129.54 90)
+    (property "Footprint" "Resistor_SMD:R_0805_2012Metric" (at 154.178 129.54 90)
       (effects (font (size 1.27 1.27)) hide)
     )
@@
       (effects (font (size 1.27 1.27)) (justify left))
     )
-    (property "Footprint" "" (at 140.0048 87.63 0)
+    (property "Footprint" "Capacitor_SMD:C_0805_2012Metric" (at 140.0048 87.63 0)
       (effects (font (size 1.27 1.27)) hide)
     )
@@
       (effects (font (size 1.27 1.27)) (justify left))
     )
-    (property "Footprint" "" (at 146.3548 87.63 0)
+    (property "Footprint" "Capacitor_SMD:C_0805_2012Metric" (at 146.3548 87.63 0)
       (effects (font (size 1.27 1.27)) hide)
     )
@@
       (effects (font (size 1.27 1.27)))
     )
-    (property "Footprint" "" (at 110.998 88.9 90)
+    (property "Footprint" "Resistor_SMD:R_0805_2012Metric" (at 110.998 88.9 90)
       (effects (font (size 1.27 1.27)) hide)
     )
@@
       (effects (font (size 1.27 1.27)) (justify left))
     )
-    (property "Footprint" "" (at 223.2152 138.43 0)
+    (property "Footprint" "Capacitor_SMD:C_0805_2012Metric" (at 223.2152 138.43 0)
       (effects (font (size 1.27 1.27)) hide)
     )
@@
       (effects (font (size 1.27 1.27)) (justify left))
     )
-    (property "Footprint" "" (at 133.6548 87.63 0)
+    (property "Footprint" "Capacitor_SMD:C_0805_2012Metric" (at 133.6548 87.63 0)
       (effects (font (size 1.27 1.27)) hide)
     )
@@
       (effects (font (size 1.27 1.27)) (justify left))
     )
-    (property "Footprint" "" (at 153.9748 90.17 0)
+    (property "Footprint" "Capacitor_SMD:C_0805_2012Metric" (at 153.9748 90.17 0)
       (effects (font (size 1.27 1.27)) hide)
     )
@@
       (effects (font (size 1.27 1.27)))
     )
-    (property "Footprint" "" (at 88.138 83.82 90)
+    (property "Footprint" "Resistor_SMD:R_0805_2012Metric" (at 88.138 83.82 90)
       (effects (font (size 1.27 1.27)) hide)
     )
@@
       (effects (font (size 1.27 1.27)))
     )
-    (property "Footprint" "" (at 107.188 88.9 90)
+    (property "Footprint" "Resistor_SMD:R_0805_2012Metric" (at 107.188 88.9 90)
       (effects (font (size 1.27 1.27)) hide)
     )
@@
       (effects (font (size 1.27 1.27)))
     )
-    (property "Footprint" "" (at 103.378 88.9 90)
+    (property "Footprint" "Resistor_SMD:R_0805_2012Metric" (at 103.378 88.9 90)
       (effects (font (size 1.27 1.27)) hide)
     )
@@
       (effects (font (size 1.27 1.27)))
     )
-    (property "Footprint" "" (at 220.218 114.3 90)
+    (property "Footprint" "Resistor_SMD:R_0805_2012Metric" (at 220.218 114.3 90)
       (effects (font (size 1.27 1.27)) hide)
     )
@@
       (effects (font (size 1.27 1.27)))
     )
-    (property "Footprint" "" (at 215.138 114.3 90)
-      (effects (font (size 1.27 1.27)) hide)
-    )
+    (property "Footprint" "Resistor_SMD:R_0805_2012Metric" (at 215.138 114.3 90)
+      (effects (font (size 1.27 1.27)) hide)
+    )

Commit message: Almost-Almost PCB design. Minor improvements on copper layer Silkscreen cleanup schematic sheet cleanup (now with subsheet titles)
Other:
- title: (none) -> Addressable LED Controller
Changed lines of the file:
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@@
 (kicad_sch (version 20230121) (generator eeschema)
   (paper "A4")
+  (title_block
+    (title "Addressable LED Controller")
+    (date "2023-07-30")
+    (rev "3.0")
+    (comment 1 "Jamal Bouajjaj")
+    (comment 2 "Ethernet Physical")
+  )
   (junction (at 214.63 146.05) (diameter 0) (color 0 0 0 0)
   )

Commit message: Final Rev 3 board
Many changes that are finalization changes mostly
Parts:
- added R11: 0, Resistor_SMD:R_0805_2012Metric, symbol Device:R
Connections:
- net GND: now also R11.2
- net at J3.SH: now also R11.1
- no-connect marks 1 -> 0
Changed lines of the file:
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@@
   (junction (at 147.32 90.17) (diameter 0) (color 0 0 0 0)
   )
-  (no_connect (at 96.52 130.81))
   (wire (pts (xy 198.12 100.33) (xy 195.58 100.33))
     (stroke (width 0) (type default))
@@
     )
   )
+  (symbol (lib_id "Device:R") (at 100.33 130.81 90) (mirror x) (unit 1)
+    (in_bom yes) (on_board yes) (dnp no)
+    (property "Reference" "R11" (at 96.52 131.445 0)
+      (effects (font (size 1.27 1.27)) (justify left))
+    )
+    (property "Value" "0" (at 100.33 130.81 90)
+      (effects (font (size 1.27 1.27)))
+    )
+    (property "Footprint" "Resistor_SMD:R_0805_2012Metric" (at 100.33 129.032 90)
+      (effects (font (size 1.27 1.27)) hide)
+    )
+    (property "Datasheet" "~" (at 100.33 130.81 0)
+      (effects (font (size 1.27 1.27)) hide)
+    )
+    (pin "1")
+    (pin "2")
+    (instances
+      (project "LED_Controller"
+        (path "/c2ef8e0f-ce81-4c82-a0ca-f054c5c3745d"
+          (reference "R11") (unit 1)
+        )
+        (path "/c2ef8e0f-ce81-4c82-a0ca-f054c5c3745d/6d0223d2-791f-4988-ac9a-278fccfb0cf9"
+          (reference "R30") (unit 1)
+        )
+      )
+    )
+  )
   (symbol (lib_id "Device:R") (at 109.22 88.9 0) (mirror y) (unit 1)
     (in_bom yes) (on_board yes) (dnp no)
@@
         )
       )
+    )
+  )
+  (symbol (lib_id "power:GND") (at 104.14 130.81 0) (mirror y) (unit 1)
+    (in_bom yes) (on_board yes) (dnp no)
+    (property "Reference" "#PWR015" (at 104.14 137.16 0)
+      (effects (font (size 1.27 1.27)) hide)
+    )
+    (property "Value" "GND" (at 104.14 134.62 0)
+      (effects (font (size 1.27 1.27)))
+    )
+    (property "Footprint" "" (at 104.14 130.81 0)
+      (effects (font (size 1.27 1.27)) hide)
+    )
+    (property "Datasheet" "" (at 104.14 130.81 0)
+      (effects (font (size 1.27 1.27)) hide)
+    )
+    (pin "1")
+    (instances
+      (project "LED_Controller"
+        (path "/c2ef8e0f-ce81-4c82-a0ca-f054c5c3745d"
+          (reference "#PWR015") (unit 1)
+        )
+        (path "/c2ef8e0f-ce81-4c82-a0ca-f054c5c3745d/6d0223d2-791f-4988-ac9a-278fccfb0cf9"
+          (reference "#PWR038") (unit 1)
+        )
+      )
