File: PCB/LED_Controller.kicad_pcb (KiCad board)
At the start: 2 copper layers, 48.3 x 58.4 mm, 45 parts, among them J1 Conn_01x04_Female, J2 Conn_01x06_Female, J3 Conn_01x06_Female, J4 Add. LED Strip, J5 Add. LED Strip, J7 Conn_01x02, Q1 MMBF170, Q10 BC817, Q2 MMBF170, Q3 MMBF170, Q4 MMBF170, Q9 BC817, SW1 SW_Push, SW2 SW_Push, U1 ESP32-WROOM-32, U2 NCP1117-5.0_SOT223, U3 NCP1117-3.3_SOT223

Commit message: Rev 2.0 local push
Parts:
- removed J3: Conn_01x06_Female, Connector_PinHeader_2.54mm:PinHeader_2x03_P2.54mm_Vertical
- removed J5: Add. LED Strip, TerminalBlock_Phoenix:TerminalBlock_Phoenix_MKDS-1,5-4-5.08_1x04_P5.08mm_Horizontal
- removed JP3: Jumper_2_Bridged, Jumper:SolderJumper-2_P1.3mm_Bridged2Bar_Pad1.0x1.5mm
- removed JP4: Jumper_3_Bridged12, Jumper:SolderJumper-3_P1.3mm_Bridged2Bar12_Pad1.0x1.5mm
- removed Q1, Q2, Q3, Q4: MMBF170, Package_TO_SOT_SMD:SOT-23
- removed Q10, Q9: BC817, Package_TO_SOT_SMD:SOT-23
- removed R10, R11, R12, R13, R19, R20, R5, R6, R8, R9: 10k, Resistor_SMD:R_0805_2012Metric_Pad1.20x1.40mm_HandSolder
- removed SW1, SW2: SW_Push, Button_Switch_SMD:SW_Push_1P1T_NO_CK_KMR2
- added AE1: Antenna_Chip, RF_Antenna:Johanson_2450AT43F0100, F.Cu at (156.6, 55.9)
- added C10: C, Capacitor_SMD:C_0805_2012Metric_Pad1.18x1.45mm_HandSolder, F.Cu at (161.7, 62.7)
- added C11: C, Capacitor_SMD:C_0805_2012Metric_Pad1.18x1.45mm_HandSolder, F.Cu at (161.7, 60.2)
- added C9: 0.1u, Capacitor_SMD:C_0603_1608Metric, F.Cu at (163.7, 65.5)
- added G***: LOGO, LOGO, F.Cu at (168.9, 57.1)
- added JP1: Jumper_2_Bridged, Jumper:SolderJumper-2_P1.3mm_Bridged2Bar_Pad1.0x1.5mm, F.Cu at (179.1, 66.7)
- added L1: 3.3uH, Inductor_SMD:L_1206_3216Metric_Pad1.22x1.90mm_HandSolder, F.Cu at (169.0, 68.3)
- added L2: L, Inductor_SMD:L_0805_2012Metric_Pad1.05x1.20mm_HandSolder, F.Cu at (158.6, 61.5)
- added U4: 74LVCH2T45DC, Package_SO:VSSOP-8_2.3x2mm_P0.5mm, F.Cu at (143.9, 63.6)
- C1: value 10uF -> 0.1uF
- C2: value 0.1uF -> 22uF; footprint Capacitor_SMD:C_0805_2012Metric_Pad1.18x1.45mm_HandSolder -> Capacitor_SMD:C_1206_3216Metric_Pad1.33x1.80mm_HandSolder
- C5: footprint Capacitor_SMD:C_0805_2012Metric_Pad1.18x1.45mm_HandSolder -> Capacitor_SMD:C_1206_3216Metric_Pad1.33x1.80mm_HandSolder
- J1: value Conn_01x04_Female -> Barrel_Jack; footprint Connector_PinHeader_2.54mm:PinHeader_2x02_P2.54mm_Vertical -> Connector_BarrelJack:BarrelJack_Horizontal
- R4: value 10k -> 31.6k
- U1: value ESP32-WROOM-32 -> ESP32-PICO-D4; footprint RF_Module:ESP32-WROOM-32 -> Package_DFN_QFN:QFN-48-1EP_7x7mm_P0.5mm_EP5.3x5.3mm
- U2: value NCP1117-5.0_SOT223 -> AP62200; footprint Package_TO_SOT_SMD:SOT-223-3_TabPin2 -> Package_TO_SOT_SMD:SOT-563
- U3: value NCP1117-3.3_SOT223 -> NCP1117-5.0_SOT223
- moved H1 61.2 mm to (183.5, 74.2)
- moved J7 60.0 mm to (193.0, 74.9), turned to 90 degrees
- moved U3 55.4 mm to (178.5, 60.5), turned to 90 degrees
- moved U2 48.8 mm to (171.9, 69.6), turned to 0 degrees
- moved C4 43.4 mm to (177.4, 71.4), turned to -90 degrees
- moved C5 42.2 mm to (168.8, 63.0), turned to 90 degrees
- moved J1 41.3 mm to (185.5, 61.3), turned to 180 degrees
- moved C3 39.8 mm to (174.9, 71.4), turned to -90 degrees
- moved G*** 35.1 mm to (181.6, 67.3)
- moved J2 35.0 mm to (171.6, 74.9)
- moved C1 34.8 mm to (171.3, 72.1), turned to 180 degrees
- moved R7 34.2 mm to (166.4, 72.1), turned to 0 degrees
- moved C2 32.4 mm to (165.7, 68.3), turned to -90 degrees
- moved R4 29.8 mm to (172.4, 65.0)
- moved H2 27.9 mm to (146.1, 57.8)
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Connections:
- C1 pad 1: +5V -> Net-(C1-Pad1)
- C1 pad 2: GND -> Net-(C1-Pad2)
- C2 pad 1: +5V -> +3V3
- C7 pad 1: VLED -> VIN
- C8 pad 1: VLED -> VIN
- J1 pad 1: /SCL -> VIN
- J1 pad 2: /SDA -> GND
- J1 pad 3: +3V3 -> (no net)
- J2 pad 2: /TX -> Net-(J2-Pad2)
- J2 pad 4: /PROG_DTR -> /EN
- J2 pad 5: /PROG_RTS -> /GPIO0
- J4 pad 4: VLED -> VIN
- R1 pad 1: +3V3 -> GND
- R1 pad 2: /LED1-DATA_{L} -> Net-(R1-Pad2)
- R4 pad 1: +5V -> Net-(R1-Pad2)
- R4 pad 2: /LED1-DATA_{H} -> +3V3
- R7 pad 1: Net-(R7-Pad1) -> /TX
- R7 pad 2: /TX -> Net-(J2-Pad2)
- U1 pad 1: GND -> +3V3
- U1 pad 10: /LED2-CLK_{L} -> /MIC_WS
- U1 pad 11: /LED2-DATA_{L} -> /MIC_SD
- U1 pad 12: /LED1-CLK_{L} -> unconnected-(U1-Pad12)
- U1 pad 13: /LED1-DATA_{L} -> /MIC_SCK
- U1 pad 14: /SCL -> unconnected-(U1-Pad14)
- U1 pad 15: GND -> unconnected-(U1-Pad15)
- U1 pad 16: /SDA -> /LED1-CLK_{L}
- U1 pad 17: unconnected-(U1-Pad17) -> /LED1-DATA_{L}
- U1 pad 19: unconnected-(U1-Pad19) -> +3V3
- U1 pad 2: +3V3 -> Net-(C10-Pad1)
- U1 pad 23: unconnected-(U1-Pad23) -> /GPIO0
- U1 pad 25: /GPIO0 -> unconnected-(U1-Pad25)
- U1 pad 26: unconnected-(U1-Pad26) -> +3V3
- U1 pad 3: /EN -> +3V3
- U1 pad 34: /RX -> unconnected-(U1-Pad34)
- U1 pad 35: Net-(R7-Pad1) -> unconnected-(U1-Pad35)
- U1 pad 37: unconnected-(U1-Pad37) -> +3V3
- U1 pad 38: GND -> unconnected-(U1-Pad38)
- U1 pad 39: GND -> unconnected-(U1-Pad39)
- U1 pad 4: unconnected-(U1-Pad4) -> +3V3
- U1 pad 6: /MIC_WS -> unconnected-(U1-Pad6)
- U1 pad 7: /MIC_SD -> unconnected-(U1-Pad7)
- U1 pad 9: /MIC_SCK -> /EN
- U2 pad 1: GND -> VIN
- U2 pad 2: +5V -> Net-(C1-Pad2)
- U2 pad 3: VIN -> GND
- U3 pad 2: +3V3 -> +5V
- U3 pad 3: +5V -> VIN
Routing:
- net +3V3: track 177.2 -> 76.8 mm
- net VIN: track 6.17 -> 78.9 mm, vias 0 -> 9
- net VLED: track 54.1 -> 0.00 mm
- net /EN: track 42.9 -> 21.1 mm, vias 3 -> 1
- net /MIC_SD: track 18.6 -> 0.00 mm
- net /MIC_SCK: track 17.8 -> 0.00 mm
- net /LED1-CLK_{L}: track 26.9 -> 11.1 mm, vias 2 -> 0
- net /PROG_RTS: track 14.4 -> 0.00 mm, vias 1 -> 0
- net /MIC_WS: track 13.9 -> 0.00 mm
- net +5V: track 80.4 -> 66.9 mm, vias 6 -> 3
- net /GPIO0: track 24.6 -> 12.9 mm
- net /LED2-CLK_{L}: track 11.5 -> 0.00 mm
- net /LED2-CLK_{H}: track 11.4 -> 0.00 mm
- net Net-(R7-Pad1): track 11.3 -> 0.00 mm
- net /LED2-DATA_{H}: track 11.2 -> 0.00 mm
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- added copper zone on F.Cu, net +3V3
- added copper zone on B.Cu, net VIN
- removed copper zone on F.Cu, net +5V
Other:
- board size 48.3 x 58.4 mm -> 66.5 x 24.1 mm
- board text added: "Rev 2"
- board text removed: "Rev 1"

Commit message: Started on board layout
Parts:
- removed J7: Conn_01x02, TerminalBlock_Phoenix:TerminalBlock_Phoenix_MKDS-1,5-2-5.08_1x02_P5.08mm_Horizontal
- added C12: 1uF, Capacitor_SMD:C_0805_2012Metric, F.Cu at (134.3, 207.4)
- added C13: 1uF, Capacitor_SMD:C_0805_2012Metric, F.Cu at (130.2, 207.4)
- added C14: 1uF, Capacitor_SMD:C_0805_2012Metric, F.Cu at (136.6, 207.4)
- added C15: 1uF, Capacitor_SMD:C_0805_2012Metric, F.Cu at (142.1, 203.4)
- added C16: 1uF, Capacitor_SMD:C_0805_2012Metric, F.Cu at (123.3, 197.7)
- added C17: C, Capacitor_SMD:C_0805_2012Metric, F.Cu at (145.9, 207.2)
- added C18: C, Capacitor_SMD:C_0805_2012Metric, F.Cu at (141.1, 211.9)
- added C19: 0.1u, Capacitor_SMD:C_0805_2012Metric, F.Cu at (53.9, 151.9)
- added C20: 330uF, Capacitor_SMD:C_Elec_6.3x5.4, F.Cu at (91.4, 109.2)
- added C21: 0.1u, Capacitor_SMD:C_Elec_6.3x5.4, F.Cu at (91.4, 117.1)
- added C22: 100uF, Capacitor_SMD:C_Elec_6.3x5.4, F.Cu at (45.7, 116.8)
- added C23: 100uF, Capacitor_SMD:C_Elec_6.3x5.8, F.Cu at (45.7, 108.5)
- added C24: 1uF, Capacitor_SMD:C_1206_3216Metric_Pad1.33x1.80mm_HandSolder, F.Cu at (45.7, 122.9)
- added C25: 0.1u, Capacitor_SMD:C_0805_2012Metric, F.Cu at (45.7, 125.7)
- added D1: SMF15A, Diode_SMD:D_SMF, F.Cu at (105.2, 149.6)
- added D2: CDBHM220L, Package_TO_SOT_SMD:TO-269AA, F.Cu at (53.3, 158.8)
- added D3: SMAJ58A, Diode_SMD:D_SMA, F.Cu at (53.9, 148.6)
- added D4: CDBHM220L, Package_TO_SOT_SMD:TO-269AA, F.Cu at (53.3, 165.4)
- added F1: Polyfuse, Fuse:Fuse_1206_3216Metric, F.Cu at (111.8, 151.4)
- added J3: 74984104400, ProjectFootprints:74984104400, F.Cu at (67.3, 171.4)
- added J5: Screw_Terminal_01x04, TerminalBlock_Phoenix:TerminalBlock_Phoenix_MKDS-1,5-4-5.08_1x04_P5.08mm_Horizontal, F.Cu at (140.6, 111.3)
- added L3: 3.3uH, Inductor_SMD:L_1206_3216Metric_Pad1.22x1.90mm_HandSolder, F.Cu at (109.5, 140.2)
- added L4: L_Ferrite, Inductor_SMD:L_0805_2012Metric, F.Cu at (132.2, 207.5)
- added L5: L_Ferrite, Inductor_SMD:L_0805_2012Metric, F.Cu at (126.4, 197.7)
- added Q1: MMBF170, Package_TO_SOT_SMD:SOT-23, F.Cu at (50.9, 140.9)
- added R10: 49.9, Resistor_SMD:R_0805_2012Metric, F.Cu at (126.4, 195.0)
- added R11: 49.9, Resistor_SMD:R_0805_2012Metric, F.Cu at (126.4, 191.1)
- added R12: 10k, Resistor_SMD:R_0805_2012Metric, F.Cu at (136.6, 196.0)
- added R13: 10k, Resistor_SMD:R_0805_2012Metric, F.Cu at (138.6, 196.0)
- added R14: 12.1k, Resistor_SMD:R_0805_2012Metric, F.Cu at (132.2, 203.4)
- added R15: R, Resistor_SMD:R_0805_2012Metric, F.Cu at (52.2, 143.9)
- added R16: R, Resistor_SMD:R_0805_2012Metric, F.Cu at (55.8, 143.9)
- added R17: R, Resistor_SMD:R_0805_2012Metric, F.Cu at (64.4, 139.2)
- added R18: R, Resistor_SMD:R_0805_2012Metric, F.Cu at (64.4, 137.2)
- added R19: R, Resistor_SMD:R_0805_2012Metric, F.Cu at (59.5, 143.9)
- added R20: 0, Resistor_SMD:R_0805_2012Metric, F.Cu at (53.4, 136.6)
- added R21: R, Resistor_SMD:R_0805_2012Metric, F.Cu at (64.4, 143.3)
- added R22: R, Resistor_SMD:R_0805_2012Metric, F.Cu at (93.5, 122.9)
- added R23: 10k, Resistor_SMD:R_0805_2012Metric, F.Cu at (134.6, 134.2)
- added R24: R, Resistor_SMD:R_0805_2012Metric, F.Cu at (64.4, 135.1)
- added R25: R, Resistor_SMD:R_0805_2012Metric, F.Cu at (64.4, 141.2)
- added R26: R, Resistor_SMD:R_0805_2012Metric, F.Cu at (89.4, 122.9)
- added R27: 10k, Resistor_SMD:R_0805_2012Metric, F.Cu at (134.6, 131.2)
- added R28: 10k, Resistor_SMD:R_0805_2012Metric, F.Cu at (134.6, 128.3)
- added R29: 0, Resistor_SMD:R_0805_2012Metric, F.Cu at (59.4, 133.3)
- added R5: 1k, Resistor_SMD:R_0805_2012Metric, F.Cu at (57.4, 175.0)
- added R6: 1k, Resistor_SMD:R_0805_2012Metric, F.Cu at (77.5, 175.0)
- added R8: 49.9, Resistor_SMD:R_0805_2012Metric, F.Cu at (126.2, 204.4)
- added R9: 49.9, Resistor_SMD:R_0805_2012Metric, F.Cu at (126.2, 200.5)
- added U5: LAN8720A, Package_DFN_QFN:VQFN-24-1EP_4x4mm_P0.5mm_EP2.5x2.5mm_ThermalVias, F.Cu at (137.1, 201.4)
- added U6: MCP1792x-5002xCB, Package_TO_SOT_SMD:SOT-23, F.Cu at (316.0, 38.6)
- added U7: VCB4805SBO-50WR3, ProjectFootprints:VCB4805SBO-50WR3, F.Cu at (54.6, 114.3)
- added Y1: ECS-250-20-33-CKM-TR, Crystal:Crystal_SMD_3225-4Pin_3.2x2.5mm, F.Cu at (143.4, 209.5)
- C10: value C -> 2.2pF; footprint Capacitor_SMD:C_0805_2012Metric_Pad1.18x1.45mm_HandSolder -> Capacitor_SMD:C_0805_2012Metric
- C11: value C -> 4pF; footprint Capacitor_SMD:C_0805_2012Metric_Pad1.18x1.45mm_HandSolder -> Capacitor_SMD:C_0805_2012Metric
- C2: value 22uF -> 0.1uF; footprint Capacitor_SMD:C_1206_3216Metric_Pad1.33x1.80mm_HandSolder -> Capacitor_SMD:C_0805_2012Metric_Pad1.18x1.45mm_HandSolder
- C4: value 0.1uF -> 10uF; footprint Capacitor_SMD:C_0805_2012Metric_Pad1.18x1.45mm_HandSolder -> Capacitor_SMD:C_1206_3216Metric_Pad1.33x1.80mm_HandSolder
- C5: value 10uF -> 22uF
- C6, C8: footprint Capacitor_SMD:C_0805_2012Metric_Pad1.18x1.45mm_HandSolder -> Capacitor_SMD:C_0805_2012Metric
- C9: footprint Capacitor_SMD:C_0603_1608Metric -> Capacitor_SMD:C_0805_2012Metric
- J4: value Add. LED Strip -> Screw_Terminal_01x02; footprint TerminalBlock_Phoenix:TerminalBlock_Phoenix_MKDS-1,5-4-5.08_1x04_P5.08mm_Horizontal -> TerminalBlock_Phoenix:TerminalBlock_Phoenix_MKDS-1,5-2-5.08_1x02_P5.08mm_Horizontal
- L1: value 3.3uH -> L_Ferrite; footprint Inductor_SMD:L_1206_3216Metric_Pad1.22x1.90mm_HandSolder -> Inductor_SMD:L_0805_2012Metric
- L2: value L -> 2.2nH
- R1: value 10k -> 31.6k
- R4: value 31.6k -> 10k
- R7: footprint Resistor_SMD:R_0805_2012Metric_Pad1.20x1.40mm_HandSolder -> Resistor_SMD:R_0805_2012Metric
- U3: value NCP1117-5.0_SOT223 -> TPS2372; footprint Package_TO_SOT_SMD:SOT-223-3_TabPin2 -> Package_DFN_QFN:Texas_S-PVQFN-N20_EP3.15x3.15mm
- moved U3 143.3 mm to (58.7, 139.2)
- moved JP1 141.8 mm to (317.1, 34.5), turned to 0 degrees
- moved J1 131.8 mm to (106.7, 167.0), turned to 90 degrees
- moved J4 122.2 mm to (88.9, 171.4), turned to 0 degrees
- moved U2 102.2 mm to (102.1, 144.3)
- moved R1 99.5 mm to (115.3, 142.7), turned to 0 degrees
- moved R4 98.8 mm to (115.3, 145.7), turned to 0 degrees
- moved C6 98.7 mm to (100.1, 136.9), turned to 0 degrees
- moved L1 97.7 mm to (118.9, 152.1), turned to 0 degrees
- moved C2 96.9 mm to (102.1, 141.5), turned to 0 degrees
- moved C1 96.6 mm to (107.7, 144.8), turned to 0 degrees
- moved C3 96.2 mm to (101.4, 133.3), turned to 0 degrees
- moved C5 93.1 mm to (107.0, 132.6), turned to 0 degrees
- moved C4 91.2 mm to (107.0, 129.2), turned to 0 degrees
- moved C11 90.3 mm to (144.9, 149.0), turned to -90 degrees
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Connections:
- net /MIC_SCK renamed /E_MDIO
- net /MIC_SD renamed /E_RXER
- net /MIC_WS renamed /E_~{INT}
- C1 pad 2: Net-(C1-Pad2) -> Net-(U2-SW)
- C2 pad 1: +3V3 -> VLED
- C3 pad 1: VIN -> VLED
- C4 pad 1: VIN -> +3V3
- C7 pad 1: VIN -> VLED
- C8 pad 1: VIN -> VLED
- J4 pad 1: /LED1-CLK_{H} -> GND
- J4 pad 2: GND -> VIN
- L1 pad 1: Net-(C1-Pad2) -> Net-(D1-A1)
- L1 pad 2: +3V3 -> VLED
- R1 pad 1: GND -> Net-(U2-FB)
- R1 pad 2: Net-(R1-Pad2) -> +3V3
- R4 pad 1: Net-(R1-Pad2) -> GND
- R4 pad 2: +3V3 -> Net-(U2-FB)
- U1 pad 12: unconnected-(U1-Pad12) -> /E_MDC
- U1 pad 14: unconnected-(U1-Pad14) -> /E_RXD0
- U1 pad 15: unconnected-(U1-Pad15) -> /E_RXD1
- U1 pad 16: /LED1-CLK_{L} -> /E_CRS
- U1 pad 18: unconnected-(U1-Pad18) -> /LED1-CLK_{L}
- U1 pad 28: unconnected-(U1-Pad28) -> /POE_TPH
- U1 pad 29: unconnected-(U1-Pad29) -> /POE_~{BT}
- U1 pad 34: unconnected-(U1-Pad34) -> /POE_TPL
- U1 pad 36: unconnected-(U1-Pad36) -> /E_~{RST}
- U1 pad 38: unconnected-(U1-Pad38) -> /E_TXD0
- U1 pad 39: unconnected-(U1-Pad39) -> /E_TXD1
- U1 pad 42: unconnected-(U1-Pad42) -> /E_TXEN
- U2 pad 1: VIN -> VLED
- U2 pad 2: Net-(C1-Pad2) -> Net-(U2-SW)
- U2 pad 5: VIN -> VLED
- U2 pad 6: Net-(R1-Pad2) -> Net-(U2-FB)
- U3 pad 1: GND -> Net-(D2-+)
- U3 pad 2: +5V -> Net-(U3-DEN)
- U3 pad 3: VIN -> Net-(U3-CLSA)
Routing:
- net VIN: track 78.9 -> 0.00 mm, vias 9 -> 0
- net +5V: track 66.9 -> 0.00 mm, vias 3 -> 0
- net +3V3: track 76.8 -> 39.3 mm, vias 8 -> 5
- net /EN: track 21.1 -> 6.55 mm, vias 1 -> 0
- net /LED1-DATA_{L}: track 11.1 -> 0.00 mm
- net /LED1-CLK_{L}: track 11.1 -> 0.00 mm
- net /LED1-CLK_{H}: track 9.14 -> 0.00 mm
- net /LED1-DATA_{H}: track 9.03 -> 0.00 mm
- net /RX: track 7.84 -> 0.00 mm
- net Net-(R1-Pad2): track 6.26 -> 0.00 mm
- net Net-(C1-Pad2): track 5.23 -> 0.00 mm
- net /TX: track 4.49 -> 0.00 mm
- net Net-(U2-BST): track 2.13 -> 0.00 mm
- net GND: track 3.15 -> 2.57 mm, vias 15 -> 5
- removed copper zone on F.Cu, net +3V3
- removed copper zone on B.Cu, net GND
- removed copper zone on F.Cu, net GND
- removed copper zone on B.Cu, net VIN
- removed copper zone on F.Cu, net VIN
Other:
- board outline removed
- board text added: "Rev 3"
- board text removed: "Rev 2"

Commit message: Started serious board layout
Parts:
- added C26: 0.1u, Capacitor_SMD:C_0805_2012Metric, F.Cu at (121.2, 160.8)
- added C27: 0.1u, Capacitor_SMD:C_0805_2012Metric, F.Cu at (126.0, 174.8)
- added H3: MountingHole_Pad, MountingHole:MountingHole_3.2mm_M3_DIN965_Pad, F.Cu at (97.5, 175.0)
- J2: footprint Connector_PinHeader_2.54mm:PinHeader_1x06_P2.54mm_Horizontal -> Connector:Tag-Connect_TC2030-IDC-NL_2x03_P1.27mm_Vertical
- R22, R26: moved to B.Cu
- U2: value AP62200 -> AP62200WU-7; footprint Package_TO_SOT_SMD:SOT-563 -> Package_TO_SOT_SMD:TSOT-23-6
- moved JP1 228.6 mm to (120.0, 150.2), turned to -90 degrees
- moved U6 228.3 mm to (116.8, 150.2), turned to 90 degrees
- moved H2 195.6 mm to (56.6, 174.2)
- moved R7 137.6 mm to (121.2, 175.8), turned to -90 degrees
- moved J2 136.1 mm to (131.5, 180.9), turned to 180 degrees
- moved H1 108.2 mm to (134.5, 121.8)
- moved J4 61.4 mm to (126.5, 122.9), turned to 180 degrees
- moved R28 60.6 mm to (114.5, 185.4), turned to 90 degrees
- moved R11 57.6 mm to (80.2, 156.7), turned to -90 degrees
- moved R27 56.2 mm to (119.8, 185.4), turned to 90 degrees
- moved R10 56.0 mm to (83.0, 159.5), turned to 180 degrees
- moved Y1 54.6 mm to (107.8, 168.2)
- moved C17 54.6 mm to (110.2, 165.8)
- moved C18 54.6 mm to (105.4, 170.6)
- moved R23 54.1 mm to (117.2, 185.4), turned to 90 degrees
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Connections:
- C2 pad 1: VLED -> Net-(U2-EN)
- C3 pad 1: VLED -> Net-(U2-EN)
- C7 pad 1: VLED -> VIN
- C8 pad 1: VLED -> VIN
- J5 pad 1: VLED -> VIN
- L1 pad 2: VLED -> Net-(U2-EN)
- R12 pad 2: /Ethernet and Connector/E_~{RST} -> /E_~{RST}
- R13 pad 2: /Ethernet and Connector/E_~{INT} -> /E_~{INT}
- U2 pad 1: VLED -> GND
- U2 pad 3: GND -> Net-(U2-EN)
- U2 pad 4: Net-(U2-BST) -> Net-(U2-FB)
- U2 pad 5: VLED -> Net-(U2-EN)
- U2 pad 6: Net-(U2-FB) -> Net-(U2-BST)
- U3 pad 17: /POE and External Power/POE_TPL -> /POE_TPH
- U3 pad 18: /POE and External Power/POE_TPH -> /POE_~{BT}
- U3 pad 19: /POE and External Power/POE_~{BT} -> /POE_TPL
- U4 pad 2: /LED1-DATA_{L} -> /LED1-CLK_{L}
- U4 pad 3: /LED1-CLK_{L} -> /LED1-DATA_{L}
- U4 pad 6: /LED1-CLK_{H} -> /LED1-DATA_{H}
- U4 pad 7: /LED1-DATA_{H} -> /LED1-CLK_{H}
- U5 pad 10: /Ethernet and Connector/E_RXER -> /E_RXER
- U5 pad 11: /Ethernet and Connector/E_CRS -> /E_CRS
- U5 pad 12: /Ethernet and Connector/E_MDIO -> /E_MDIO
- U5 pad 13: /Ethernet and Connector/E_MDC -> /E_MDC
- U5 pad 14: /Ethernet and Connector/E_~{INT} -> /E_~{INT}
- U5 pad 15: /Ethernet and Connector/E_~{RST} -> /E_~{RST}
- U5 pad 16: /Ethernet and Connector/E_TXEN -> /E_TXEN
- U5 pad 17: /Ethernet and Connector/E_TXD0 -> /E_TXD0
- U5 pad 18: /Ethernet and Connector/E_TXD1 -> /E_TXD1
- U5 pad 7: /Ethernet and Connector/E_RXD1 -> /E_RXD1
- U5 pad 8: /Ethernet and Connector/E_RXD0 -> /E_RXD0
Routing:
- net +3V3: track 39.3 -> 110.9 mm, vias 5 -> 10
- net /Ethernet and Connector/ETH_RX-: track 0.00 -> 35.6 mm
- net /LED1-CLK_{H}: track 0.00 -> 33.6 mm
- net Net-(J3-CD): track 0.00 -> 33.3 mm, vias 0 -> 4
- net /Ethernet and Connector/ETH_RX+: track 0.00 -> 32.7 mm
- net /POE_TPL: track 0.00 -> 30.0 mm, vias 0 -> 1
- net /Ethernet and Connector/ETH_TX-: track 0.00 -> 29.3 mm
- net /POE_TPH: track 0.00 -> 29.0 mm, vias 0 -> 1
- net /POE_~{BT}: track 0.00 -> 28.9 mm, vias 0 -> 1
- net Net-(D2-+): track 0.00 -> 28.8 mm
- net /Ethernet and Connector/ETH_TX+: track 0.00 -> 27.5 mm
- net Net-(U3-PG): track 0.00 -> 23.1 mm, vias 0 -> 1
- net /LED1-DATA_{H}: track 0.00 -> 22.0 mm
- net Vdda2: track 0.00 -> 19.5 mm, vias 0 -> 2
- net /Ethernet and Connector/ETH_V1+: track 0.00 -> 14.8 mm
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- added copper zone on B.Cu, net GND
- added copper zone on F.Cu, net GND
- added copper zone on F.Cu, net Net-(D2-+)
- added copper zone on B.Cu, net Net-(D2--)
- added copper zone on F.Cu, net Net-(D2--)
- added copper zone on F.Cu, net Net-(U7-GND)
- added copper zone on F.Cu, net VIN
Other:
- board outline added: 89.5 x 60.5 mm

Commit message: More layout work
Parts:
- moved R27 25.6 mm to (113.5, 160.6), turned to 180 degrees
- moved R23 22.7 mm to (113.5, 163.0), turned to 180 degrees
- moved R28 20.2 mm to (113.5, 165.2), turned to 180 degrees
- moved R13 17.5 mm to (111.7, 173.0), turned to 45 degrees
- moved R12 14.2 mm to (113.1, 174.4), turned to 45 degrees
- moved R7 8.13 mm to (127.0, 181.5)
- moved C8 3.64 mm to (124.5, 146.8), turned to -135 degrees
- moved H3 1.82 mm to (99.2, 174.5)
- moved Y1 1.31 mm to (106.6, 168.8)
- moved C17 1.28 mm to (109.0, 166.3)
- moved C18 1.28 mm to (104.2, 171.0)
- moved C9 1.27 mm to (117.5, 175.0)
- moved U4 1.06 mm to (128.0, 159.8)
- moved C12 0.67 mm to (100.0, 167.0)
- moved C13 0.67 mm to (95.9, 167.0)
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Connections:
- U1 pad 10: /E_~{INT} -> unconnected-(U1-IO34-Pad10)
- U1 pad 11: /E_RXER -> /LED1-DATA_{L}
- U1 pad 12: /E_MDC -> /LED1-CLK_{L}
- U1 pad 13: /E_MDIO -> /E_RXER
- U1 pad 17: /LED1-DATA_{L} -> unconnected-(U1-IO14-Pad17)
- U1 pad 18: /LED1-CLK_{L} -> unconnected-(U1-IO12-Pad18)
- U1 pad 25: unconnected-(U1-IO16-Pad25) -> /POE_TPH
- U1 pad 27: unconnected-(U1-IO17-Pad27) -> /POE_~{BT}
- U1 pad 28: /POE_TPH -> /POE_TPL
- U1 pad 29: /POE_~{BT} -> /E_MDIO
- U1 pad 34: /POE_TPL -> /E_MDC
- U1 pad 35: unconnected-(U1-IO18-Pad35) -> /E_~{INT}
Routing:
- net +3V3: track 110.9 -> 184.9 mm, vias 10 -> 14
- net VIN: track 4.24 -> 57.5 mm
- net /Ethernet and Connector/ETH_LED2: track 0.00 -> 46.9 mm, vias 0 -> 2
- net /POE_TPH: track 29.0 -> 74.2 mm, vias 1 -> 2
- net /POE_~{BT}: track 28.9 -> 73.8 mm, vias 1 -> 2
- net /POE_TPL: track 30.0 -> 72.5 mm, vias 1 -> 2
- net /Ethernet and Connector/ETH_LED1: track 0.00 -> 31.7 mm, vias 0 -> 2
- net /E_TXEN: track 11.1 -> 39.8 mm, vias 0 -> 2
- net /E_~{INT}: track 9.21 -> 35.9 mm, vias 0 -> 2
- net /E_TXD0: track 11.8 -> 37.7 mm, vias 0 -> 2
- net /E_TXD1: track 12.9 -> 37.8 mm, vias 0 -> 2
- net /E_~{RST}: track 10.1 -> 32.7 mm, vias 0 -> 2
- net /E_CRS: track 7.77 -> 29.0 mm, vias 0 -> 2
- net /E_RXER: track 7.77 -> 28.9 mm
- net /E_RXD0: track 7.43 -> 28.2 mm
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
Commit message: Close-to-final PCB layout, passes most routing DRC I think
Parts:
- moved J2 25.7 mm to (106.3, 175.9), turned to 0 degrees
- moved R7 21.1 mm to (108.2, 171.8), turned to -135 degrees
- moved H2 4.11 mm to (52.5, 174.5)
- moved C11 2.26 mm to (130.7, 174.0)
- moved C10 2.25 mm to (128.3, 174.0)
- moved L2 1.90 mm to (129.5, 170.6)
- moved C27 1.25 mm to (125.5, 175.9), turned to -45 degrees
- moved H3 1.25 mm to (98.0, 174.5)
- moved L3 1.00 mm to (103.5, 150.0)
- moved C9 0.90 mm to (116.8, 174.5)
- moved H1 0.56 mm to (134.0, 122.0)
- moved AE1 0.30 mm to (135.5, 173.4)
- moved C4 0.25 mm to (107.6, 149.2)
- moved C5 0.25 mm to (110.1, 149.2)
Routing:
- net +3V3: track 184.9 -> 228.5 mm, vias 14 -> 15
- net /GPIO0: track 3.46 -> 40.8 mm, vias 0 -> 2
- net /EN: track 2.98 -> 34.7 mm, vias 0 -> 2
- net /TX: track 0.00 -> 21.7 mm
- net GND: track 9.66 -> 30.7 mm
- net /RX: track 0.00 -> 20.8 mm, vias 0 -> 2
- net Net-(AE1-FEED): track 0.00 -> 7.32 mm
- net /Ethernet and Connector/ETH_TX+: track 27.4 -> 34.3 mm
- net /Ethernet and Connector/ETH_TX-: track 29.2 -> 36.0 mm
- net Net-(U1-LNA_IN): track 0.00 -> 5.97 mm
- net Net-(J2-Pin_2): track 0.00 -> 3.91 mm
- net Net-(U7-GND): track 0.00 -> 3.54 mm
- net Net-(U2-EN): track 10.0 -> 13.0 mm
- net +5V: track 17.4 -> 15.6 mm
- net Net-(U2-SW): track 8.86 -> 7.47 mm
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