File: PCB/LED_Controller.kicad_sch (KiCad schematic)
At the start: 20 parts, among them J2 Conn_01x06_Female, J5 Screw_Terminal_01x04, U1 ESP32-PICO-D4, U4 74LVCH2T45DC

Commit message: More layout work
Connections:
- net E_MDC: now also U1.34 (IO5); no longer U1.12 (IO32)
- net E_MDIO: now also U1.29 (SD3/IO10); no longer U1.13 (IO33)
- net E_RXER: now also U1.13 (IO33); no longer U1.11 (IO35)
- net E_~{INT}: now also U1.35 (IO18); no longer U1.10 (IO34)
- net LED1-CLK_{L}: now also U1.12 (IO32); no longer U1.18 (IO12)
- net LED1-DATA_{L}: now also U1.11 (IO35); no longer U1.17 (IO14)
- net POE_TPH: now also U1.25 (IO16); no longer U1.28 (SD2/IO9)
- net POE_TPL: now also U1.28 (SD2/IO9); no longer U1.34 (IO5)
- net POE_~{BT}: now also U1.27 (IO17); no longer U1.29 (SD3/IO10)
- no-connect marks 7 -> 5
Changed lines of the file:
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@@
   (no_connect (at 40.64 146.05))
   (no_connect (at 40.64 148.59))
-  (no_connect (at 40.64 138.43))
   (no_connect (at 40.64 151.13))
   (no_connect (at 116.84 102.87))
-  (no_connect (at 40.64 140.97))
   (no_connect (at 40.64 143.51))
   (wire (pts (xy 69.85 49.53) (xy 59.69 49.53))
@@
     (stroke (width 0) (type solid))
   )
+  (wire (pts (xy 34.29 140.97) (xy 40.64 140.97))
+    (stroke (width 0) (type default))
+  )
   (wire (pts (xy 69.85 54.61) (xy 59.69 54.61))
     (stroke (width 0) (type default))
@@
     (stroke (width 0) (type default))
   )
-  (wire (pts (xy 91.44 151.13) (xy 81.28 151.13))
-    (stroke (width 0) (type default))
-  )
-  (wire (pts (xy 91.44 166.37) (xy 81.28 166.37))
+  (wire (pts (xy 81.28 138.43) (xy 91.44 138.43))
+    (stroke (width 0) (type default))
+  )
+  (wire (pts (xy 95.25 151.13) (xy 81.28 151.13))
+    (stroke (width 0) (type default))
+  )
+  (wire (pts (xy 96.52 166.37) (xy 81.28 166.37))
     (stroke (width 0) (type default))
   )
@@
     (stroke (width 0) (type default))
   )
+  (wire (pts (xy 34.29 138.43) (xy 40.64 138.43))
+    (stroke (width 0) (type default))
+  )
   (wire (pts (xy 182.88 156.21) (xy 182.88 161.29))
     (stroke (width 0) (type default))
@@
     (stroke (width 0) (type solid))
   )
-  (wire (pts (xy 91.44 143.51) (xy 81.28 143.51))
+  (wire (pts (xy 95.25 143.51) (xy 81.28 143.51))
     (stroke (width 0) (type default))
   )
@@
     (stroke (width 0) (type default))
   )
-  (wire (pts (xy 81.28 163.83) (xy 91.44 163.83))
+  (wire (pts (xy 81.28 163.83) (xy 96.52 163.83))
     (stroke (width 0) (type default))
   )
@@
     (stroke (width 0) (type solid))
   )
-  (wire (pts (xy 91.44 153.67) (xy 81.28 153.67))
+  (wire (pts (xy 95.25 153.67) (xy 81.28 153.67))
     (stroke (width 0) (type default))
   )
@@
     (stroke (width 0) (type default))
   )
-  (wire (pts (xy 91.44 156.21) (xy 81.28 156.21))
-    (stroke (width 0) (type default))
-  )
-  (wire (pts (xy 81.28 128.27) (xy 96.52 128.27))
-    (stroke (width 0) (type solid))
+  (wire (pts (xy 95.25 156.21) (xy 81.28 156.21))
+    (stroke (width 0) (type default))
   )
   (wire (pts (xy 180.34 156.21) (xy 180.34 158.75))
@@
     (stroke (width 0) (type solid))
   )
-  (wire (pts (xy 91.44 158.75) (xy 81.28 158.75))
+  (wire (pts (xy 96.52 158.75) (xy 81.28 158.75))
     (stroke (width 0) (type default))
   )
@@
     (stroke (width 0) (type default))
   )
-  (wire (pts (xy 81.28 133.35) (xy 96.52 133.35))
-    (stroke (width 0) (type solid))
-  )
   (wire (pts (xy 59.69 64.77) (xy 69.85 64.77))
     (stroke (width 0) (type default))
@@
     (stroke (width 0) (type solid))
   )
-  (wire (pts (xy 91.44 140.97) (xy 81.28 140.97))
+  (wire (pts (xy 95.25 140.97) (xy 81.28 140.97))
     (stroke (width 0) (type default))
   )
@@
     (stroke (width 0) (type solid))
   )
-  (wire (pts (xy 91.44 146.05) (xy 81.28 146.05))
+  (wire (pts (xy 95.25 146.05) (xy 81.28 146.05))
     (stroke (width 0) (type default))
   )
@@
     (effects (font (size 1.27 1.27)) (justify left bottom))
   )
-  (label "E_MDC" (at 91.44 158.75 180) (fields_autoplaced)
+  (label "E_MDC" (at 91.44 120.65 180) (fields_autoplaced)
     (effects (font (size 1.27 1.27)) (justify right bottom))
   )
@@
     (effects (font (size 1.27 1.27)) (justify left bottom))
   )
-  (label "E_RXD0" (at 91.44 151.13 180) (fields_autoplaced)
-    (effects (font (size 1.27 1.27)) (justify right bottom))
-  )
-  (label "E_TXD0" (at 91.44 140.97 180) (fields_autoplaced)
+  (label "E_RXD0" (at 95.25 151.13 180) (fields_autoplaced)
+    (effects (font (size 1.27 1.27)) (justify right bottom))
+  )
+  (label "E_TXD0" (at 95.25 140.97 180) (fields_autoplaced)
     (effects (font (size 1.27 1.27)) (justify right bottom))
   )
@@
     (effects (font (size 1.27 1.27)) (justify left bottom))
   )
-  (label "E_RXER" (at 91.44 166.37 180) (fields_autoplaced)
-    (effects (font (size 1.27 1.27)) (justify right bottom))
-  )
-  (label "POE_TPL" (at 91.44 120.65 180) (fields_autoplaced)
+  (label "E_RXER" (at 91.44 161.29 180) (fields_autoplaced)
+    (effects (font (size 1.27 1.27)) (justify right bottom))
+  )
+  (label "POE_TPL" (at 91.44 123.19 180) (fields_autoplaced)
     (effects (font (size 1.27 1.27)) (justify right bottom))
   )
@@
     (effects (font (size 1.27 1.27)) (justify left bottom))
   )
-  (label "POE_~{BT}" (at 91.44 125.73 180) (fields_autoplaced)
-    (effects (font (size 1.27 1.27)) (justify right bottom))
+  (label "POE_~{BT}" (at 34.29 140.97 0) (fields_autoplaced)
+    (effects (font (size 1.27 1.27)) (justify left bottom))
   )
   (label "E_TXEN" (at 69.85 44.45 180) (fields_autoplaced)
@@
     (effects (font (size 1.27 1.27)) (justify right bottom))
   )
-  (label "E_RXD1" (at 91.44 153.67 180) (fields_autoplaced)
+  (label "E_RXD1" (at 95.25 153.67 180) (fields_autoplaced)
     (effects (font (size 1.27 1.27)) (justify right bottom))
   )
@@
     (effects (font (size 1.27 1.27)) (justify right bottom))
   )
-  (label "LED1-CLK_{L}" (at 96.52 128.27 180) (fields_autoplaced)
-    (effects (font (size 1.27 1.27)) (justify right bottom))
-  )
-  (label "E_MDIO" (at 91.44 161.29 180) (fields_autoplaced)
-    (effects (font (size 1.27 1.27)) (justify right bottom))
-  )
-  (label "E_TXD1" (at 91.44 146.05 180) (fields_autoplaced)
+  (label "LED1-CLK_{L}" (at 96.52 158.75 180) (fields_autoplaced)
+    (effects (font (size 1.27 1.27)) (justify right bottom))
+  )
+  (label "E_MDIO" (at 91.44 125.73 180) (fields_autoplaced)
+    (effects (font (size 1.27 1.27)) (justify right bottom))
+  )
+  (label "E_TXD1" (at 95.25 146.05 180) (fields_autoplaced)
     (effects (font (size 1.27 1.27)) (justify right bottom))
   )
@@
     (effects (font (size 1.27 1.27)) (justify left bottom))
   )
-  (label "E_CRS" (at 91.44 156.21 180) (fields_autoplaced)
+  (label "E_CRS" (at 95.25 156.21 180) (fields_autoplaced)
     (effects (font (size 1.27 1.27)) (justify right bottom))
   )
@@
     (effects (font (size 1.27 1.27)) (justify right bottom))
   )
-  (label "LED1-DATA_{L}" (at 96.52 133.35 180) (fields_autoplaced)
+  (label "LED1-DATA_{L}" (at 96.52 166.37 180) (fields_autoplaced)
     (effects (font (size 1.27 1.27)) (justify right bottom))
   )
@@
     (effects (font (size 1.27 1.27)) (justify right bottom))
   )
-  (label "POE_TPH" (at 91.44 123.19 180) (fields_autoplaced)
-    (effects (font (size 1.27 1.27)) (justify right bottom))
+  (label "POE_TPH" (at 34.29 138.43 0) (fields_autoplaced)
+    (effects (font (size 1.27 1.27)) (justify left bottom))
   )
   (label "POE_~{BT}" (at 168.91 158.75 0) (fields_autoplaced)
@@
     (effects (font (size 1.27 1.27)) (justify right bottom))
   )
-  (label "E_TXEN" (at 91.44 143.51 180) (fields_autoplaced)
+  (label "E_TXEN" (at 95.25 143.51 180) (fields_autoplaced)
     (effects (font (size 1.27 1.27)) (justify right bottom))
   )
@@
     (effects (font (size 1.27 1.27)) (justify right bottom))
   )
-  (label "E_~{INT}" (at 91.44 163.83 180) (fields_autoplaced)
-    (effects (font (size 1.27 1.27)) (justify right bottom))
-  )
+  (label "E_~{INT}" (at 91.44 138.43 180) (fields_autoplaced)
+    (effects (font (size 1.27 1.27)) (justify right bottom))
+  )

Commit message: Final Rev 3 board
Many changes that are finalization changes mostly
Parts:
- C10, C11: footprint Capacitor_SMD:C_0805_2012Metric -> Capacitor_SMD:C_0603_1608Metric
- L2: footprint Inductor_SMD:L_0805_2012Metric_Pad1.05x1.20mm_HandSolder -> Inductor_SMD:L_0603_1608Metric
Other:
- sheet POE and External Power ports: added none; removed POE_DIS
Changed lines of the file:
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@@
     (effects (font (size 1.27 1.27)) (justify right bottom))
+  )
+  (netclass_flag "" (length 2.54) (shape round) (at 68.58 34.29 0) (fields_autoplaced)
+    (effects (font (size 1.27 1.27)) (justify left bottom))
+    (property "Netclass" "HI_V" (at 69.469 31.75 0)
+      (effects (font (size 1.27 1.27) italic) (justify left))
+    )
+  )
+  (netclass_flag "" (length 2.54) (shape round) (at 71.12 36.83 0) (fields_autoplaced)
+    (effects (font (size 1.27 1.27)) (justify left bottom))
+    (property "Netclass" "HI_V" (at 72.009 34.29 0)
+      (effects (font (size 1.27 1.27) italic) (justify left))
+    )
+  )
+  (netclass_flag "" (length 2.54) (shape round) (at 66.04 31.75 0) (fields_autoplaced)
+    (effects (font (size 1.27 1.27)) (justify left bottom))
+    (property "Netclass" "HI_V" (at 66.929 29.21 0)
+      (effects (font (size 1.27 1.27) italic) (justify left))
+    )
+  )
+  (netclass_flag "" (length 2.54) (shape round) (at 63.5 29.21 0) (fields_autoplaced)
+    (effects (font (size 1.27 1.27)) (justify left bottom))
+    (property "Netclass" "HI_V" (at 64.389 26.67 0)
+      (effects (font (size 1.27 1.27) italic) (justify left))
+    )
   )
   (symbol (lib_id "power:GND") (at 165.1 179.07 0) (unit 1)
@@
       (effects (font (size 1.27 1.27)) (justify left))
     )
-    (property "Footprint" "Capacitor_SMD:C_0805_2012Metric" (at 97.4852 110.49 0)
+    (property "Footprint" "Capacitor_SMD:C_0603_1608Metric" (at 97.4852 110.49 0)
       (effects (font (size 1.27 1.27)) hide)
     )
@@
       (effects (font (size 1.27 1.27)))
     )
-    (property "Footprint" "Inductor_SMD:L_0805_2012Metric_Pad1.05x1.20mm_HandSolder" (at 102.87 102.87 0)
+    (property "Footprint" "Inductor_SMD:L_0603_1608Metric" (at 102.87 102.87 0)
       (effects (font (size 1.27 1.27)) hide)
     )
@@
       (effects (font (size 1.27 1.27)) (justify left))
     )
-    (property "Footprint" "Capacitor_SMD:C_0805_2012Metric" (at 110.1852 110.49 0)
+    (property "Footprint" "Capacitor_SMD:C_0603_1608Metric" (at 110.1852 110.49 0)
       (effects (font (size 1.27 1.27)) hide)
     )
@@
       (effects (font (size 1.27 1.27)) (justify left))
     )
-    (pin "POE_DIS" input (at 121.92 38.1 0)
-      (effects (font (size 1.27 1.27)) (justify right))
-    )
     (pin "POE_TPH" output (at 121.92 27.94 0)

Commit message: Updated to Rev 4
Parts:
- removed H1, H2, H3: MountingHole_Pad, MountingHole:MountingHole_3.2mm_M3_DIN965_Pad, symbol Mechanical:MountingHole_Pad
- removed J5: Screw_Terminal_01x04, TerminalBlock_Phoenix:TerminalBlock_Phoenix_MKDS-1,5-4-5.08_1x04_P5.08mm_Horizontal, symbol Connector:Screw_Terminal_01x04
- removed R23, R27, R28: 10k, Resistor_SMD:R_0805_2012Metric, symbol Device:R
- added C1, C2, C6, C8: 0.1uF, Capacitor_SMD:C_0603_1608Metric, symbol Device:C
- added C17: 0.1u, Capacitor_SMD:C_0603_1608Metric, symbol Device:C_Small
- added C3, C5: 22uF, Capacitor_SMD:C_1206_3216Metric_Pad1.33x1.80mm_HandSolder, symbol Device:C
- added D1: SMF15A, Diode_SMD:D_SMF, symbol Diode:SMF15A
- added D2: SP0505BAHT, Package_TO_SOT_SMD:SOT-23-6, symbol Power_Protection:SP0505BAHT
- added F1: Polyfuse, Fuse:Fuse_1206_3216Metric, symbol Device:Polyfuse
- added J1: Barrel_Jack, Connector_BarrelJack:BarrelJack_Horizontal, symbol Connector:Barrel_Jack
- added J3: Screw_Terminal_01x02, TerminalBlock_Phoenix:TerminalBlock_Phoenix_MKDS-1,5-2-5.08_1x02_P5.08mm_Horizontal, symbol Connector:Screw_Terminal_01x02
- added J5: LED Data Out, TerminalBlock_Phoenix:TerminalBlock_Phoenix_PT-1,5-2-3.5-H_1x02_P3.50mm_Horizontal, symbol Connector:Screw_Terminal_01x02
- added J6: LED Data Out, TerminalBlock_TE-Connectivity:TerminalBlock_TE_282834-4_1x04_P2.54mm_Horizontal, symbol Connector:Screw_Terminal_01x04
- added JP1: Jumper_2_Bridged, Jumper:SolderJumper-2_P1.3mm_Open_TrianglePad1.0x1.5mm, symbol Jumper:Jumper_2_Open
- added L1: L_Ferrite, Inductor_SMD:L_0805_2012Metric, symbol Device:L_Ferrite
- added L3: 3.3uH, Inductor_SMD:L_1206_3216Metric_Pad1.22x1.90mm_HandSolder, symbol Device:L
- added R1: 31.6k, Resistor_SMD:R_0805_2012Metric_Pad1.20x1.40mm_HandSolder, symbol Device:R
- added R4: 10k, Resistor_SMD:R_0805_2012Metric_Pad1.20x1.40mm_HandSolder, symbol Device:R
- added U2: AP62200WU-7, Package_TO_SOT_SMD:TSOT-23-6, symbol ProjectLibrary:AP62200WU-7
- added U3: 74LVCH2T45DC, Package_SO:VSSOP-8_2.3x2mm_P0.5mm, symbol Logic_LevelTranslator:74LVCH2T45DC
- added U5: MCP1792x-5002xCB, Package_TO_SOT_SMD:SOT-23, symbol Regulator_Linear:MCP1792x-5002xCB
- C10: value 2.2pF -> 3.9pF
- C11: value 4pF -> 4.3pF
- C26, C27, C9: footprint Capacitor_SMD:C_0805_2012Metric -> Capacitor_SMD:C_0603_1608Metric
- L2: value 2.2nH -> 2.3nH
- R2, R3: footprint Resistor_SMD:R_0805_2012Metric_Pad1.20x1.40mm_HandSolder -> Resistor_SMD:R_0603_1608Metric
- R7: footprint Resistor_SMD:R_0805_2012Metric -> Resistor_SMD:R_0603_1608Metric_Pad0.98x0.95mm_HandSolder
Connections:
- net +3V3: now also J2.3 (Pin_3), C17.1, C5.1, C6.1, L3.2, R1.2, U3.1 (VCCA), U3.5 (DIR); no longer J2.1 (Pin_1)
- net +5V: now also JP1.2 (B), U3.8 (VCCB), U5.2 (VO)
- net GND: now also C17.2, C2.2, C3.2, C5.2, C6.2, C8.2, D1.2 (A2), D2.2 (A), J1.2, J3.1 (Pin_1), J5.1 (Pin_1), R4.1, U2.1 (GND), U3.4 (GND), U5.1 (GND)
- net LED1-CLK_{H}: now also D2.5 (K), J6.4 (Pin_4)
- net LED1-CLK_{L}: now also U1.20 (IO13); no longer U1.12 (IO32)
- net LED1-DATA_{H}: now also D2.6 (K), J6.3 (Pin_3)
- net LED1-DATA_{L}: now also U1.21 (IO15); no longer U1.11 (IO35)
- net RX: now also J2.1 (Pin_1); no longer J2.3 (Pin_3)
- net LED2-CLK_{L}: now reaches U1.17 (IO14)
- net LED2-CLK_{L}: now also U3.2 (1A)
- net LED2-DATA_{L}: now reaches U1.18 (IO12)
- net LED2-DATA_{L}: now also U3.3 (2A)
- net E_CRS: no longer names the net of U1.16 (IO27)
- net E_MDC: no longer names the net of U1.34 (IO5)
- net E_MDIO: no longer names the net of U1.29 (SD3/IO10)
- net E_RXD0: no longer names the net of U1.14 (IO25)
- net E_RXD1: no longer names the net of U1.15 (IO26)
- net E_RXER: no longer names the net of U1.13 (IO33)
- net E_TXD0: no longer names the net of U1.38 (IO19)
- net E_TXD1: no longer names the net of U1.39 (IO22)
- net E_TXEN: no longer names the net of U1.42 (IO21)
- net E_~{INT}: no longer names the net of U1.35 (IO18)
- net E_~{RST}: no longer names the net of U1.36 (IO23)
- net POE_TPH: no longer names the net of U1.25 (IO16)
- net POE_TPL: no longer names the net of U1.28 (SD2/IO9)
- net POE_~{BT}: no longer names the net of U1.27 (IO17)
- new net: R1.1, R4.2, U2.4 (FB)
- new net: C2.1, C3.1, L1.2, U2.3 (VIN), U2.5 (EN)
- new net: D1.1 (A1), F1.2, L1.1
- new net: C1.2, L3.1, U2.2 (SW)
- new net: C1.1, U2.6 (BST)
- new net LED2-CLK_{H}: D2.1 (K), J6.2 (Pin_2), U3.7 (1B)
- new net LED2-DATA_{H}: D2.3 (K), J6.1 (Pin_1), U3.6 (2B)
- new net VIN: C8.1, F1.1, J1.1, J3.2 (Pin_2), J5.2 (Pin_2), JP1.1 (A), U5.3 (VI)
- no-connect marks 5 -> 15
Other:
- removed sheet Ethernet and Connector
- removed sheet POE and External Power
- note removed: "Pins that can be swapped/moved E_RST E_MDC E_MDOI E_INT E_RXER LED1-CLK_{L} LED1-DATA_{L} POE_~{BT} POE_TPH POE_TPL"
- moved on the sheet: AE1, C10, C11, C26, C27, C9, J2, L2, R2, R3, R7, U1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
